File: Current Meter V1/currentSensor.kicad_sch (KiCad schematic)
At the start: 17 parts, among them U201 A1308xLHxx-1, U202 MCP6002-xSN

Commit message: microcontroller update
Parts:
- renumbered C205 to C801, C206 to C802, C201 to C803, C207 to C804, C208 to C805, D201 to D801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
