File: Current Meter V1/buck.kicad_sch (KiCad schematic)
At the start: 13 parts, among them SW1 SW_DIP_x01, U2 TPS5430DDAR

Commit message: buck
Parts:
- removed C1, C6: 100u, Capacitor_THT:CP_Radial_D8.0mm_P3.50mm, symbol bfr_capacitors:50ZLH100MEFC8X11.5
- removed C2: 10u, Capacitor_SMD:C_0603_1608Metric, symbol bfr_capacitors:CL05A106MQ5NUNC
- removed C3, C5: 100n, Capacitor_SMD:C_0402_1005Metric_Pad0.74x0.62mm_HandSolder, symbol bfr_capacitors:CL05B104KB54PNC
- removed C7: 220u, Capacitor_THT:CP_Radial_D8.0mm_P3.50mm, symbol bfr_capacitors:35ZLH220MEFC8X11.5
- removed R3: 100k, Resistor_SMD:R_0402_1005Metric_Pad0.72x0.64mm_HandSolder, symbol bfr_resistors:RMCF0402FT100K
- removed R4: 51k, Resistor_SMD:R_0402_1005Metric_Pad0.72x0.64mm_HandSolder, symbol bfr_resistors:RMCF0402FT51K0
- removed R6: 10k, Resistor_SMD:R_0402_1005Metric_Pad0.72x0.64mm_HandSolder, symbol bfr_resistors:RMCF0402FT10K0
- added C1: 10u, Capacitor_SMD:C_0603_1608Metric_Pad1.08x0.95mm_HandSolder, symbol bfr_capacitors:CL10A106MA8NRNC
- added C2: 10n, Capacitor_SMD:C_0603_1608Metric_Pad1.08x0.95mm_HandSolder, symbol bfr_capacitors:VJ0603Y103KXAAC
- added C3: 220u, Capacitor_THT:CP_Radial_D8.0mm_P3.50mm, symbol bfr_capacitors:35ZLH220MEFC8X11.5
- added R1: 10k, Resistor_SMD:R_0805_2012Metric_Pad1.20x1.40mm_HandSolder, symbol bfr_resistors:RMCF0805FT10K0
- added R2: 3.3k, Resistor_SMD:R_0805_2012Metric_Pad1.20x1.40mm_HandSolder, symbol bfr_resistors:RMCF0805FT3K30
- L1: footprint Inductor_SMD:L_6.3x6.3_H3 -> bfr_inductors:CDRH104RNP-150NC
Connections:
- net +5_V: now also C3.1, R1.2
- net GND: now also C1.2, C3.2, R2.1
- net SW_NODE: now also C2.2
- net VIN: now also C1.1
- net at U2.4 (VSENSE): now also R1.1, R2.2
- net at U2.1 (BOOT): now also C2.1

Commit message: changed everything to 5V
Parts:
- renumbered C1 to C601, C2 to C602, C3 to C603, D1 to D601, L1 to L601, R1 to R601, R2 to R602, SW1 to SW601, U2 to U601
Changed lines of the file:
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@@
 		(dnp no)
 		(fields_autoplaced yes)
-		(property "Reference" "R2"
+		(property "Reference" "R602"
 			(at 220.98 110.4899 90)
 			(effects
@@
 			(project ""
 				(path "/a2a38fd0-928e-4aba-88ec-c7bc808fdbf7/46638e6b-22d6-417c-82d4-58dcfaa6d532"
-					(reference "R2")
+					(reference "R602")
 					(unit 1)
 				)
@@
 		(dnp no)
 		(fields_autoplaced yes)
-		(property "Reference" "#PWR?"
+		(property "Reference" "#PWR0603"
 			(at 134.62 101.6 0)
 			(effects
@@
 			(project "CMU - Current Measurement Unit"
 				(path "/a2a38fd0-928e-4aba-88ec-c7bc808fdbf7/46638e6b-22d6-417c-82d4-58dcfaa6d532"
-					(reference "#PWR?")
+					(reference "#PWR0603")
 					(unit 1)
 				)
@@
 		(dnp no)
 		(fields_autoplaced yes)
-		(property "Reference" "L1"
+		(property "Reference" "L601"
 			(at 194.31 67.31 0)
 			(effects
@@
 			(project ""
 				(path "/a2a38fd0-928e-4aba-88ec-c7bc808fdbf7/46638e6b-22d6-417c-82d4-58dcfaa6d532"
-					(reference "L1")
+					(reference "L601")
 					(unit 1)
 				)
@@
 		(dnp no)
 		(fields_autoplaced yes)
-		(property "Reference" "D1"
+		(property "Reference" "D601"
 			(at 181.61 80.9624 90)
 			(effects
@@
 			(project ""
 				(path "/a2a38fd0-928e-4aba-88ec-c7bc808fdbf7/46638e6b-22d6-417c-82d4-58dcfaa6d532"
-					(reference "D1")
+					(reference "D601")
 					(unit 1)
 				)
@@
 		(dnp no)
 		(fields_autoplaced yes)
-		(property "Reference" "SW1"
+		(property "Reference" "SW601"
 			(at 123.19 96.52 0)
 			(effects
@@
 			(project "CMU - Current Measurement Unit"
 				(path "/a2a38fd0-928e-4aba-88ec-c7bc808fdbf7/46638e6b-22d6-417c-82d4-58dcfaa6d532"
-					(reference "SW1")
+					(reference "SW601")
 					(unit 1)
 				)
@@
 		(dnp no)
 		(fields_autoplaced yes)
-		(property "Reference" "#PWR01"
+		(property "Reference" "#PWR0604"
 			(at 179.07 100.33 0)
 			(effects
@@
 			(project ""
 				(path "/a2a38fd0-928e-4aba-88ec-c7bc808fdbf7/46638e6b-22d6-417c-82d4-58dcfaa6d532"
-					(reference "#PWR01")
+					(reference "#PWR0604")
 					(unit 1)
 				)
@@
 		(dnp no)
 		(fields_autoplaced yes)
-		(property "Reference" "#PWR?"
+		(property "Reference" "#PWR0602"
 			(at 130.81 115.57 0)
 			(effects
@@
 			(project "CMU - Current Measurement Unit"
 				(path "/a2a38fd0-928e-4aba-88ec-c7bc808fdbf7/46638e6b-22d6-417c-82d4-58dcfaa6d532"
-					(reference "#PWR?")
+					(reference "#PWR0602")
 					(unit 1)
 				)
@@
 		(dnp no)
 		(fields_autoplaced yes)
-		(property "Reference" "C1"
+		(property "Reference" "C601"
 			(at 106.68 74.9299 0)
 			(effects
@@
 			(project ""
 				(path "/a2a38fd0-928e-4aba-88ec-c7bc808fdbf7/46638e6b-22d6-417c-82d4-58dcfaa6d532"
-					(reference "C1")
+					(reference "C601")
 					(unit 1)
 				)
@@
 		(dnp no)
 		(fields_autoplaced yes)
-		(property "Reference" "#PWR02"
+		(property "Reference" "#PWR0605"
 			(at 205.74 100.33 0)
 			(effects
@@
 			(project ""
 				(path "/a2a38fd0-928e-4aba-88ec-c7bc808fdbf7/46638e6b-22d6-417c-82d4-58dcfaa6d532"
-					(reference "#PWR02")
+					(reference "#PWR0605")
 					(unit 1)
 				)
@@
 		(dnp no)
 		(fields_autoplaced yes)
-		(property "Reference" "#PWR03"
+		(property "Reference" "#PWR0606"
 			(at 218.44 127 0)
 			(effects
@@
 			(project ""
 				(path "/a2a38fd0-928e-4aba-88ec-c7bc808fdbf7/46638e6b-22d6-417c-82d4-58dcfaa6d532"
-					(reference "#PWR03")
+					(reference "#PWR0606")
 					(unit 1)
 				)
@@
 		(dnp no)
 		(fields_autoplaced yes)
-		(property "Reference" "C2"
+		(property "Reference" "C602"
 			(at 161.29 64.77 90)
 			(effects
@@
 			(project ""
 				(path "/a2a38fd0-928e-4aba-88ec-c7bc808fdbf7/46638e6b-22d6-417c-82d4-58dcfaa6d532"
-					(reference "C2")
+					(reference "C602")
 					(unit 1)
 				)
@@
 		(dnp no)
 		(fields_autoplaced yes)
-		(property "Reference" "C3"
+		(property "Reference" "C603"
 			(at 209.55 78.1049 0)
 			(effects
@@
 			(project ""
 				(path "/a2a38fd0-928e-4aba-88ec-c7bc808fdbf7/46638e6b-22d6-417c-82d4-58dcfaa6d532"
-					(reference "C3")
+					(reference "C603")
 					(unit 1)
 				)
@@
 		(dnp no)
 		(fields_autoplaced yes)
-		(property "Reference" "#PWR?"
+		(property "Reference" "#PWR0601"
 			(at 102.87 93.98 0)
 			(effects
@@
 			(project "CMU - Current Measurement Unit"
 				(path "/a2a38fd0-928e-4aba-88ec-c7bc808fdbf7/46638e6b-22d6-417c-82d4-58dcfaa6d532"
-					(reference "#PWR?")
+					(reference "#PWR0601")
 					(unit 1)
 				)
@@
 		(dnp no)
 		(fields_autoplaced yes)
-		(property "Reference" "R1"
+		(property "Reference" "R601"
 			(at 220.98 80.0099 90)
 			(effects
@@
 			(project ""
 				(path "/a2a38fd0-928e-4aba-88ec-c7bc808fdbf7/46638e6b-22d6-417c-82d4-58dcfaa6d532"
-					(reference "R1")
+					(reference "R601")
 					(unit 1)
 				)
@@
 		(dnp no)
 		(fields_autoplaced yes)
-		(property "Reference" "U?"
+		(property "Reference" "U601"
 			(at 135.89 64.77 0)
 			(effects
@@
 			(project "CMU - Current Measurement Unit"
 				(path "/a2a38fd0-928e-4aba-88ec-c7bc808fdbf7/46638e6b-22d6-417c-82d4-58dcfaa6d532"
-					(reference "U?")
-					(unit 1)
-				)
+					(reference "U601")
+					(unit 1)
+				)

Commit message: updated layout
Parts:
- removed SW601: SW_DIP_x01, Button_Switch_SMD:SW_DIP_SPSTx01_Slide_6.7x4.1mm_W6.73mm_P2.54mm_LowProfile_JPin, symbol Switch:SW_DIP_x01
Connections:
- net VIN renamed +12_V
- no-connect marks 0 -> 1
Changed lines of the file:
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@@
 		(color 0 0 0 0)
 	)
+	(no_connect
+		(at 123.19 82.55)
+	)
 	(wire
 		(pts
@@
 	(wire
 		(pts
-			(xy 115.57 82.55) (xy 123.19 82.55)
-		)
-		(stroke
-			(width 0)
-			(type default)
-		)
-	)
-	(wire
-		(pts
 			(xy 133.35 87.63) (xy 133.35 92.71)
 		)
@@
 	(wire
 		(pts
-			(xy 115.57 82.55) (xy 115.57 104.14)
-		)
-		(stroke
-			(width 0)
-			(type default)
-		)
-	)
-	(wire
-		(pts
 			(xy 135.89 87.63) (xy 135.89 92.71)
 		)
@@
 		(pts
 			(xy 205.74 83.82) (xy 205.74 93.98)
-		)
-		(stroke
-			(width 0)
-			(type default)
-		)
-	)
-	(wire
-		(pts
-			(xy 130.81 104.14) (xy 130.81 109.22)
 		)
 		(stroke
@@
 		)
 	)
-	(hierarchical_label "VIN"
+	(hierarchical_label "+12_V"
 		(shape input)
 		(at 88.9 72.39 180)
@@
 		(dnp no)
 		(fields_autoplaced yes)
-		(property "Reference" "#PWR0603"
+		(property "Reference" "#PWR0602"
 			(at 134.62 101.6 0)
 			(effects
@@
 			(project "CMU - Current Measurement Unit"
 				(path "/a2a38fd0-928e-4aba-88ec-c7bc808fdbf7/46638e6b-22d6-417c-82d4-58dcfaa6d532"
-					(reference "#PWR0603")
+					(reference "#PWR0602")
 					(unit 1)
 				)
@@
 	)
 	(symbol
-		(lib_id "Switch:SW_DIP_x01")
-		(at 123.19 104.14 0)
-		(unit 1)
-		(exclude_from_sim no)
-		(in_bom yes)
-		(on_board yes)
-		(dnp no)
-		(fields_autoplaced yes)
-		(property "Reference" "SW601"
-			(at 123.19 96.52 0)
-			(effects
-				(font
-					(size 1.27 1.27)
-				)
-			)
-		)
-		(property "Value" "SW_DIP_x01"
-			(at 123.19 99.06 0)
-			(effects
-				(font
-					(size 1.27 1.27)
-				)
-			)
-		)
-		(property "Footprint" "Button_Switch_SMD:SW_DIP_SPSTx01_Slide_6.7x4.1mm_W6.73mm_P2.54mm_LowProfile_JPin"
-			(at 123.19 104.14 0)
-			(effects
-				(font
-					(size 1.27 1.27)
-				)
-				(hide yes)
-			)
-		)
-		(property "Datasheet" "~"
-			(at 123.19 104.14 0)
-			(effects
-				(font
-					(size 1.27 1.27)
-				)
-				(hide yes)
-			)
-		)
-		(property "Description" "1x DIP Switch, Single Pole Single Throw (SPST) switch, small symbol"
-			(at 123.19 104.14 0)
-			(effects
-				(font
-					(size 1.27 1.27)
-				)
-				(hide yes)
-			)
-		)
-		(pin "2"
-		)
-		(pin "1"
-		)
-		(instances
-			(project "buck"
-				(path "/34dcc5f9-f36c-4889-afc0-c2fb7a9a5d2e"
-					(reference "SW1")
-					(unit 1)
-				)
-			)
-			(project "CMU - Current Measurement Unit"
-				(path "/a2a38fd0-928e-4aba-88ec-c7bc808fdbf7/46638e6b-22d6-417c-82d4-58dcfaa6d532"
-					(reference "SW601")
-					(unit 1)
-				)
-			)
-		)
-	)
-	(symbol
 		(lib_id "power:GND")
 		(at 179.07 93.98 0)
@@
 		(dnp no)
 		(fields_autoplaced yes)
-		(property "Reference" "#PWR0604"
+		(property "Reference" "#PWR0603"
 			(at 179.07 100.33 0)
 			(effects
@@
 			(project ""
 				(path "/a2a38fd0-928e-4aba-88ec-c7bc808fdbf7/46638e6b-22d6-417c-82d4-58dcfaa6d532"
-					(reference "#PWR0604")
-					(unit 1)
-				)
-			)
-		)
-	)
-	(symbol
-		(lib_id "power:GND")
-		(at 130.81 109.22 0)
-		(unit 1)
-		(exclude_from_sim no)
-		(in_bom yes)
-		(on_board yes)
-		(dnp no)
-		(fields_autoplaced yes)
-		(property "Reference" "#PWR0602"
-			(at 130.81 115.57 0)
-			(effects
-				(font
-					(size 1.27 1.27)
-				)
-				(hide yes)
-			)
-		)
-		(property "Value" "GND"
-			(at 130.81 114.3 0)
-			(effects
-				(font
-					(size 1.27 1.27)
-				)
-			)
-		)
-		(property "Footprint" ""
-			(at 130.81 109.22 0)
-			(effects
-				(font
-					(size 1.27 1.27)
-				)
-				(hide yes)
-			)
-		)
-		(property "Datasheet" ""
-			(at 130.81 109.22 0)
-			(effects
-				(font
-					(size 1.27 1.27)
-				)
-				(hide yes)
-			)
-		)
-		(property "Description" "Power symbol creates a global label with name \"GND\" , ground"
-			(at 130.81 109.22 0)
-			(effects
-				(font
-					(size 1.27 1.27)
-				)
-				(hide yes)
-			)
-		)
-		(pin "1"
-		)
-		(instances
-			(project "buck"
-				(path "/34dcc5f9-f36c-4889-afc0-c2fb7a9a5d2e"
-					(reference "#PWR06")
-					(unit 1)
-				)
-			)
-			(project "CMU - Current Measurement Unit"
-				(path "/a2a38fd0-928e-4aba-88ec-c7bc808fdbf7/46638e6b-22d6-417c-82d4-58dcfaa6d532"
-					(reference "#PWR0602")
+					(reference "#PWR0603")
 					(unit 1)
 				)
@@
 		(dnp no)
 		(fields_autoplaced yes)
-		(property "Reference" "#PWR0605"
+		(property "Reference" "#PWR0604"
 			(at 205.74 100.33 0)
 			(effects
@@
 			(project ""
 				(path "/a2a38fd0-928e-4aba-88ec-c7bc808fdbf7/46638e6b-22d6-417c-82d4-58dcfaa6d532"
-					(reference "#PWR0605")
+					(reference "#PWR0604")
 					(unit 1)
 				)
@@
 		(dnp no)
 		(fields_autoplaced yes)
-		(property "Reference" "#PWR0606"
+		(property "Reference" "#PWR0605"
 			(at 218.44 127 0)
 			(effects
@@
 			(project ""
 				(path "/a2a38fd0-928e-4aba-88ec-c7bc808fdbf7/46638e6b-22d6-417c-82d4-58dcfaa6d532"
-					(reference "#PWR0606")
+					(reference "#PWR0605")
 					(unit 1)
 				)

Commit message: added sensor connector, updated pcb layout
Parts:
- U601: footprint Package_SO:TI_SO-PowerPAD-8_ThermalVias -> Package_SO:TI_SO-PowerPAD-8
Changed lines of the file:
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@@
 			)
 		)
-		(property "Footprint" "Package_SO:TI_SO-PowerPAD-8_ThermalVias"
+		(property "Footprint" "Package_SO:TI_SO-PowerPAD-8"
 			(at 137.16 86.36 0)
 			(effects
