File: Current Meter V1/opamp.kicad_sch (KiCad schematic)
At the start: 12 parts, among them U201 MCP6002-xSN

Commit message: added sensor connector, updated pcb layout
Parts:
- TP201: footprint TestPoint:TestPoint_Keystone_5019_Miniature -> bfr_utilities:TestPoint_Keystone_5019_Miniature
Changed lines of the file:
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@@
 			)
 		)
-		(property "Footprint" "TestPoint:TestPoint_Keystone_5019_Miniature"
+		(property "Footprint" "bfr_utilities:TestPoint_Keystone_5019_Miniature"
 			(at 173.482 97.536 0)
 			(effects
