File: Current Meter V1/sensorConnector.kicad_sch (KiCad schematic)
At the start: 1 part, among them J702 Sensor Connector

Commit message: basically done board layout (hopefully)
Connections:
- net GND: no longer J702.2
- new net V_REF: J702.2
Changed lines of the file:
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@@
 	(generator_version "9.0")
 	(paper "A4")
-	(junction
-		(at 95.25 97.79)
-		(diameter 0)
-		(color 0 0 0 0)
-	)
 	(wire
 		(pts
-			(xy 95.25 97.79) (xy 95.25 105.41)
-		)
-		(stroke
-			(width 0)
-			(type default)
-		)
-	)
-	(wire
-		(pts
-			(xy 91.44 97.79) (xy 95.25 97.79)
+			(xy 88.9 105.41) (xy 100.33 105.41)
 		)
 		(stroke
@@
 	(wire
 		(pts
-			(xy 95.25 105.41) (xy 100.33 105.41)
-		)
-		(stroke
-			(width 0)
-			(type default)
-		)
-	)
-	(wire
-		(pts
-			(xy 95.25 97.79) (xy 100.33 97.79)
+			(xy 91.44 97.79) (xy 100.33 97.79)
 		)
 		(stroke
@@
 			(width 0)
 			(type default)
+		)
+	)
+	(label "V_REF"
+		(at 88.9 105.41 0)
+		(effects
+			(font
+				(size 1.27 1.27)
+			)
+			(justify left bottom)
 		)
 	)
@@
 		)
 		(pin "2"
+			(alternate "V_REF")
 		)
 		(pin "1"
