File: Current Meter V1/CMU - Current Measurement Unit.kicad_pcb (KiCad board)
At the start: 4 copper layers, 55.3 x 79.8 mm, 39 parts, among them J401 I2C OLED Display Connector, J501 Connector, J702 Sensor Connector, U201 MCP6002-xSN, U601 TPS5430DDAR

Commit message: added copper layers
Parts:
- moved G*** 10.0 mm to (153.7, 121.6)
- moved D201 5.27 mm to (127.8, 140.2)
- moved C202 3.50 mm to (127.9, 135.8), turned to -90 degrees
Routing:
- net /opamp/2.5V, 0.55V-4.5V: track 32.2 -> 23.3 mm
- net GND: track 102.1 -> 93.2 mm, vias 42 -> 46
- net +5_V: track 43.8 -> 42.0 mm, vias 14 -> 15
- net /buck/+12_V: track 57.9 -> 58.9 mm
- added copper zone on B.Cu, net GND
- added copper zone on F.Cu, net GND
- removed copper zone on F.Cu, net +5_V
